Commit message: [M-HRI] [v6]: honghai

File: assets/urdf/usb/factory_rectangular_hole_8mm.urdf (robot description, URDF)
Before this commit: robot factory_rectangular_hole_8mm, 1 links, 0 joints
Links:
- link factory_rectangular_hole_8mm: geometry collision mesh filename=factory_rectangular_hole_8mm_subdiv_3x.obj scale=2 2 5; visual mesh filename=factory_rectangular_hole_8mm_subdiv_3x.obj scale=2 2 5
