Commit message: [M-HRI][v10]:robot peg insertion finish

File: assets/urdf/peg_insertion/pentagon.urdf (robot description, URDF)
Before this commit: robot triangle, 1 links, 0 joints
Links:
- removed link triangle
- added link pentagon, mass 0.026; collision mesh filename=pentagon.obj scale=10.0 10.0 10.0; visual mesh filename=pentagon.obj scale=10.0 10.0 10.0

File: assets/urdf/peg_insertion/pentagon_kit.urdf (robot description, URDF)
Before this commit: robot triangle, 1 links, 0 joints
Links:
- removed link triangle
- added link pentagon_kit, mass 0.026; collision mesh filename=pentagon_kit.obj scale=10.0 10.0 10.0; visual mesh filename=pentagon_kit.obj scale=10.0 10.0 10.0

File: assets/urdf/peg_insertion/rectangle.urdf (robot description, URDF)
Before this commit: robot triangle, 1 links, 0 joints
Links:
- removed link triangle
- added link rectangle, mass 0.026; collision mesh filename=rectangle.obj scale=10.0 10.0 10.0; visual mesh filename=rectangle.obj scale=10.0 10.0 10.0

File: assets/urdf/peg_insertion/rectangle_kit.urdf (robot description, URDF)
Before this commit: robot triangle, 1 links, 0 joints
Links:
- removed link triangle
- added link rectangle_kit, mass 0.026; collision mesh filename=rectangle_kit.obj scale=10.0 10.0 10.0; visual mesh filename=rectangle_kit.obj scale=10.0 10.0 10.0

File: assets/urdf/peg_insertion/square.urdf (robot description, URDF)
Before this commit: robot triangle, 1 links, 0 joints
Links:
- removed link triangle
- added link square, mass 0.026; collision mesh filename=square.obj scale=10.0 10.0 10.0; visual mesh filename=square.obj scale=10.0 10.0 10.0

File: assets/urdf/peg_insertion/square_kit.urdf (robot description, URDF)
Before this commit: robot triangle, 1 links, 0 joints
Links:
- removed link triangle
- added link square_kit, mass 0.026; collision mesh filename=square_kit.obj scale=10.0 10.0 10.0; visual mesh filename=square_kit.obj scale=10.0 10.0 10.0

File: assets/urdf/peg_insertion/triangle_kit.urdf (robot description, URDF)
Before this commit: robot block_A, 1 links, 0 joints
Links:
- removed link block_A
- added link triangle_kit, mass 0.026; collision mesh filename=triangle_kit.obj scale=10.0 10.0 10.0; visual mesh filename=triangle_kit.obj scale=10.0 10.0 10.0
