Commit message: [M-HRI][v10.1]:peg insertion gen hand pose unfinish

File: assets/urdf/peg_insertion/hexagon.urdf (robot description, URDF)
Before this commit: robot pentagon, 1 links, 0 joints
Links:
- removed link pentagon
- added link hexagon, mass 0.026; collision mesh filename=hexagon.obj scale=10.0 10.0 10.0; visual mesh filename=hexagon.obj scale=10.0 10.0 10.0

File: assets/urdf/peg_insertion/pentagon_kit.urdf (robot description, URDF)
Before this commit: robot pentagon_kit, 1 links, 0 joints
Links:
- removed link pentagon_kit
- added link hexagon_kit, mass 0.026; collision mesh filename=hexagon_kit.obj scale=10.0 10.0 10.0; visual mesh filename=hexagon_kit.obj scale=10.0 10.0 10.0
